Commit message: update

File: TsenseI_hand_A3.2_withid_upper_thumb5mm_noupper_mid/urdf/TsenseI_hand_left_v3_2_withid.urdf (robot description, URDF)
Before this commit: robot TsenseI_hand_v3_2_withid_left_raised5mm, 22 links, 21 joints
Joints:
- joint left_hand_thumb_rotaback_joint2: axis 0 0 1 -> -0 -0 -1; limit lower=-1.74 upper=-0.0 effort=1.0 velocity=1.0 -> lower=0.0 upper=1.74 effort=1.0 velocity=1.0

File: TsenseI_hand_A3.2_withid_upper_thumb5mm_noupper_mid/urdf/TsenseI_hand_right_v3_2_withid.urdf (robot description, URDF)
Before this commit: robot TsenseI_hand_v3_2_withid_right_raised5mm, 22 links, 21 joints
Joints:
- joint right_hand_thumb_rotaback_joint2: axis 0 0 -1 -> -0 -0 1; limit lower=-1.74 upper=-0.0 effort=1.0 velocity=1.0 -> lower=0.0 upper=1.74 effort=1.0 velocity=1.0
